File: Hardware/Flight_Computer/RCS_Hardware.kicad_pcb (KiCad board)
At the start: 2 copper layers, 60 x 52 mm, 56 parts, among them J2 TYPE-C-31-M-12, J4 5V, J8 Conn_01x05_Male, U1 STM32F401CCU6, U2 AMS1117-3.3, U4 BNO055, U5 W25Q32JVSS, U6 MPU-6050, Y1 16MHz, Y2 32.768Mhz

Commit message: removed RCS-specific components
removed solenoid connectors, SPI connectors, LTC, and extra IMU
Parts:
- removed C21, C24: 0.1uF, Capacitor_SMD:C_0402_1005Metric
- removed C22: 2.2nF, Capacitor_SMD:C_0402_1005Metric
- removed C23: 100nF, Capacitor_SMD:C_0402_1005Metric
- removed C25: 10nF, Capacitor_SMD:C_0402_1005Metric
- removed J8: Conn_01x05_Male, Connector_PinHeader_2.54mm:PinHeader_1x05_P2.54mm_Vertical
- removed LTC: LTC1690N8, LTC1690N8:LTC1690N8
- removed SPI1, SPI2: SPI, Connector_PinHeader_2.54mm:PinHeader_1x08_P2.54mm_Vertical
- removed Solenoids: Solenoids, Connector_PinHeader_2.54mm:PinHeader_1x07_P2.54mm_Vertical
- removed U6: MPU-6050, Sensor_Motion:InvenSense_QFN-24_4x4mm_P0.5mm
- renumbered Flash to J1, Power to J5
Connections:
- U1 pad 11: /S1 -> unconnected-(U1-PA1-Pad11)
- U1 pad 12: /RX -> unconnected-(U1-PA2-Pad12)
- U1 pad 13: /TX -> unconnected-(U1-PA3-Pad13)
- U1 pad 19: /S2 -> unconnected-(U1-PB1-Pad19)
- U1 pad 21: /S3 -> unconnected-(U1-PB10-Pad21)
- U1 pad 26: /S4 -> unconnected-(U1-PB13-Pad26)
- U1 pad 27: /S5 -> unconnected-(U1-PB14-Pad27)
- U1 pad 28: /S6 -> unconnected-(U1-PB15-Pad28)
Routing:
- net GND: track 144.3 -> 99.4 mm, vias 21 -> 17
- net /MOSI2: track 36.8 -> 0.00 mm
- net /MISO2: track 31.4 -> 0.00 mm
- net /SCL: track 54.0 -> 22.8 mm, vias 2 -> 0
- net /SDA: track 55.4 -> 24.4 mm, vias 2 -> 0
- net +3.3V: track 148.9 -> 119.4 mm, vias 10 -> 8
- net VBUS: track 96.1 -> 67.8 mm, vias 1 -> 0
- net /S6: track 27.9 -> 0.00 mm
- net /S1: track 27.7 -> 0.00 mm
- net /SCK: track 25.9 -> 0.00 mm
- net /S5: track 25.6 -> 0.00 mm
- net /TX: track 23.9 -> 0.00 mm, vias 1 -> 0
- net /S4: track 23.8 -> 0.00 mm
- net /S3: track 23.0 -> 0.00 mm
- net /S2: track 22.4 -> 0.00 mm, vias 2 -> 0
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Other:
- board text removed: "3.3V"
- board text removed: "A"
- board text removed: "B"
- board text removed: "CS"
- board text removed: "MISO"
- board text removed: "MOSI"
- board text removed: "S1"
- board text removed: "S2"
- board text removed: "S3"
- board text removed: "S4"
- board text removed: "S5"
- board text removed: "S6"
- board text removed: "SCK"
- board text removed: "SCL"
- board text removed: "SDA"
- board text removed: "SPI1"
- board text removed: "SPI2"
- board text removed: "Y"
- board text removed: "Z"
