File: Hardware/Flight_Computer/_autosave-ARES_FC.kicad_sch (KiCad schematic)
At the start: 63 parts, among them J1 SWD, J2 TYPE-C-31-M-12, J3 To Motor Board, J4 5V, J5 GND, J6 To Motor Board, U1 STM32F401CCU6, U2 AMS1117-3.3, U3 BMP280, U4 BNO055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

Commit message: first pass FC changes
Connections:
- net VDD is gone; now on net +3.3V: C24.2, U3.8 (VDD)
- net +3.3V: now also C23.2, U3.6 (VDDIO)
- net CS_BMP: now reaches U1.29 (PA8)
- net CS_BMP: now also U3.2 (CSB)
- removed net VDDIO: C23.2, U3.2 (CSB), U3.6 (VDDIO)
- no-connect marks 29 -> 28

Commit message: Seperated lines that were previously merged All UART devices were on the same bus and have since been moved to GPS_UART and RADIO_UART Motor UART has been replaced with I2C NRST lines have been seperated out for motor/radio
Connections:
- net +3.3V: now also J3.5 (Pin_5), J3.6 (Pin_6), U1.21 (PB10), U1.39 (PB3); no longer C23.2, C24.2, U3.6 (VDDIO), U3.8 (VDD)
- net LED_B: now also U1.29 (PA8); no longer U1.30 (PA9)
- net NRST: no longer J3.7 (Pin_7), J6.7 (Pin_7)
- net RADIO_NRST: now reaches U1.18 (PB0)
- net RADIO_NRST: now also J6.7 (Pin_7)
- net MOTOR_NRST: now reaches U1.19 (PB1)
- net MOTOR_NRST: now also J3.7 (Pin_7)
- net RX_RADIO: now reaches U1.31 (PA10)
- net RX_RADIO: now also J6.6 (Pin_6)
- net CS_BMP renamed VDDIO
- net VDDIO: now also C23.2, U3.6 (VDDIO); no longer U1.29 (PA8)
- net RX renamed RX_GPS
- net RX_GPS: no longer J3.6 (Pin_6), J6.6 (Pin_6)
- net TX renamed TX_GPS
- net TX_GPS: no longer J3.5 (Pin_5), J6.5 (Pin_5)
- new net TX_RADIO: J6.5 (Pin_5), U1.30 (PA9)
- new net VDD: C24.2, U3.8 (VDD)
- no-connect marks 28 -> 23
Other:
- moved on the sheet: BT1, C2, C22, C3, D4, Y1

Commit message: Converted BMP280 to I2C was wrongly setup as SPI
Connections:
- net VDD: no longer names the net of C24.2, U3.8 (VDD)
- net VDDIO: no longer names the net of C23.2, U3.6 (VDDIO)
- net VDDIO: no longer U3.2 (CSB)
Changed lines of the file:
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@@
 	)
 	(junction
-		(at 316.23 60.96)
-		(diameter 0)
-		(color 0 0 0 0)
-	)
-	(junction
 		(at 87.63 135.89)
 		(diameter 0)
@@
 	)
 	(junction
-		(at 316.23 52.07)
-		(diameter 0)
-		(color 0 0 0 0)
-	)
-	(junction
 		(at 204.47 79.502)
 		(diameter 0)
@@
 		)
 	)
-	(wire
-		(pts
-			(xy 316.23 60.96) (xy 316.23 52.07)
-		)
-		(stroke
-			(width 0)
-			(type default)
-		)
-	)
 	(polyline
 		(pts
@@
 	(wire
 		(pts
-			(xy 316.23 49.53) (xy 316.23 52.07)
-		)
-		(stroke
-			(width 0)
-			(type default)
-		)
-	)
-	(wire
-		(pts
 			(xy 298.45 60.96) (xy 300.99 60.96)
 		)
@@
 	(wire
 		(pts
-			(xy 316.23 52.07) (xy 346.71 52.07)
-		)
-		(stroke
-			(width 0)
-			(type default)
-		)
-	)
-	(wire
-		(pts
 			(xy 109.22 137.16) (xy 106.68 137.16)
 		)
@@
 	(wire
 		(pts
-			(xy 308.61 60.96) (xy 316.23 60.96)
+			(xy 308.61 60.96) (xy 321.31 60.96)
 		)
 		(stroke
@@
 	(wire
 		(pts
-			(xy 321.31 60.96) (xy 316.23 60.96)
-		)
-		(stroke
-			(width 0)
-			(type default)
-		)
-	)
-	(wire
-		(pts
 			(xy 242.062 75.692) (xy 243.586 75.692)
 		)
@@
 	(wire
 		(pts
-			(xy 346.71 52.07) (xy 346.71 58.42)
-		)
-		(stroke
-			(width 0)
-			(type default)
-		)
-	)
-	(wire
-		(pts
 			(xy 364.49 133.35) (xy 368.3 133.35)
 		)
@@
 	)
 	(symbol
-		(lib_id "power:VBUS")
-		(at 316.23 49.53 0)
-		(unit 1)
-		(exclude_from_sim no)
-		(in_bom yes)
-		(on_board yes)
-		(dnp no)
-		(property "Reference" "#PWR017"
-			(at 316.23 53.34 0)
-			(effects
-				(font
-					(size 1.27 1.27)
-				)
-				(hide yes)
-			)
-		)
-		(property "Value" "VDDIO"
-			(at 316.23 45.72 0)
-			(effects
-				(font
-					(size 1.27 1.27)
-				)
-			)
-		)
-		(property "Footprint" ""
-			(at 316.23 49.53 0)
-			(effects
-				(font
-					(size 1.27 1.27)
-				)
-				(hide yes)
-			)
-		)
-		(property "Datasheet" ""
-			(at 316.23 49.53 0)
-			(effects
-				(font
-					(size 1.27 1.27)
-				)
-				(hide yes)
-			)
-		)
-		(property "Description" ""
-			(at 316.23 49.53 0)
-			(effects
-				(font
-					(size 1.27 1.27)
-				)
-				(hide yes)
-			)
-		)
-		(pin "1"
-		)
-		(instances
-			(project "ARES_FC"
-				(path "/449acbee-2eeb-4316-a8e9-c26dd430524e"
-					(reference "#PWR017")
-					(unit 1)
-				)
-			)
-		)
-	)
-	(symbol
 		(lib_id "power:GND")
 		(at 46.99 200.66 270)
@@
 					(unit 1)
 				)
-			)
-		)
-	)
-	(symbol
-		(lib_id "power:VBUS")
-		(at 312.42 53.34 0)
-		(unit 1)
-		(exclude_from_sim no)
-		(in_bom yes)
-		(on_board yes)
-		(dnp no)
-		(property "Reference" "#PWR016"
-			(at 312.42 57.15 0)
-			(effects
-				(font
-					(size 1.27 1.27)
-				)
-				(hide yes)
-			)
-		)
-		(property "Value" "VDD"
-			(at 312.42 49.53 0)
-			(effects
-				(font
-					(size 1.27 1.27)
-				)
-			)
-		)
-		(property "Footprint" ""
-			(at 312.42 53.34 0)
-			(effects
-				(font
-					(size 1.27 1.27)
-				)
-				(hide yes)
-			)
-		)
-		(property "Datasheet" ""
-			(at 312.42 53.34 0)
-			(effects
-				(font
-					(size 1.27 1.27)
-				)
-				(hide yes)
-			)
-		)
-		(property "Description" ""
-			(at 312.42 53.34 0)
-			(effects
-				(font
-					(size 1.27 1.27)
-				)
-				(hide yes)
-			)
-		)
-		(pin "1"
-		)
-		(instances
-			(project "ARES_FC"
-				(path "/449acbee-2eeb-4316-a8e9-c26dd430524e"
-					(reference "#PWR016")
-					(unit 1)
-				)
