File: Hardware/Flight_Computer/ARES_FC.kicad_sch (KiCad schematic)
At the start: 63 parts, among them J1 SWD, J2 TYPE-C-31-M-12, J3 To Motor Board, J4 5V, J5 GND, J6 To Motor Board, U1 STM32F401CCU6, U2 AMS1117-3.3, U3 BMP280, U4 BNO055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

Commit message: forgot to save everything before last commit
Connections:
- net VDD is gone; now on net +3.3V: C24.2, U3.8 (VDD)
- net VDDIO is gone; now on net +3.3V: C23.2, U3.2 (CSB), U3.6 (VDDIO)
- net +3.3V: now also J3.5 (Pin_5), J3.6 (Pin_6), U1.21 (PB10), U1.39 (PB3), U3.5 (SDO)
- net LED_B: now also U1.29 (PA8); no longer U1.30 (PA9)
- net MISO: no longer U3.5 (SDO)
- net MOSI: no longer U3.3 (SDI)
- net NRST: no longer J3.7 (Pin_7), J6.7 (Pin_7)
- net SCL: now also U3.4 (SCK)
- net SCLK: no longer U3.4 (SCK)
- net SDA: now also U3.3 (SDI)
- net RADIO_NRST: now reaches U1.18 (PB0)
- net RADIO_NRST: now also J6.7 (Pin_7)
- net MOTOR_NRST: now reaches U1.19 (PB1)
- net MOTOR_NRST: now also J3.7 (Pin_7)
- net RX_RADIO: now reaches U1.31 (PA10)
- net RX_RADIO: now also J6.6 (Pin_6)
- net RX renamed RX_GPS
- net RX_GPS: no longer J3.6 (Pin_6), J6.6 (Pin_6)
- net TX renamed TX_GPS
- net TX_GPS: no longer J3.5 (Pin_5), J6.5 (Pin_5)
- new net TX_RADIO: J6.5 (Pin_5), U1.30 (PA9)
- no-connect marks 29 -> 23
Other:
- moved on the sheet: BT1, C2, C22, C3, D4, Y1

Commit message: Routing 75% complete
added all footprints and connected most components
Parts:
- removed BT1: Battery, Battery:BatteryHolder_Keystone_103_1x20mm, symbol Device:Battery
- removed C22: 100nF, Capacitor_SMD:C_0402_1005Metric, symbol Device:C
- H1, H2, H3, H4: footprint MountingHole:MountingHole_3.2mm_M3 -> MountingHole:MountingHole_2.2mm_M2
- J3: value To Motor Board -> FC_M/P; footprint (none) -> Connector_FFC-FPC:Molex_200528-0080_1x08-1MP_P1.00mm_Horizontal
- J6: value To Motor Board -> FC_RF; footprint (none) -> Connector_FFC-FPC:Molex_200528-0080_1x08-1MP_P1.00mm_Horizontal
- U6: footprint (none) -> CD-PA1616D:XCVR_CD-PA1616D
Connections:
- net GND: now also U6.19 (GND); no longer U6.20 (NC)
- net RX_RADIO: now also J6.5 (Pin_5); no longer J6.6 (Pin_6)
- net TX_RADIO: now also J6.6 (Pin_6); no longer J6.5 (Pin_5)
- no-connect marks 23 -> 24

Commit message: routing 99% done
double check external antenna connector. S1 & S2 unused for ribbons. DRC not completed.
Connections:
- net S1 renamed S1_MP
- net S1_MP: no longer J6.3 (Pin_3)
- net S2 renamed S2_MP
- net S2_MP: no longer J6.4 (Pin_4)
- new net S1_RF: J6.3 (Pin_3)
- new net S2_RF: J6.4 (Pin_4)
Changed lines of the file:
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@@
 	(wire
 		(pts
-			(xy 69.85 187.96) (xy 73.66 187.96)
+			(xy 67.31 187.96) (xy 73.66 187.96)
 		)
 		(stroke
@@
 	(wire
 		(pts
-			(xy 44.45 190.5) (xy 48.26 190.5)
+			(xy 41.91 190.5) (xy 48.26 190.5)
 		)
 		(stroke
@@
 	(wire
 		(pts
-			(xy 44.45 187.96) (xy 48.26 187.96)
+			(xy 41.91 187.96) (xy 48.26 187.96)
 		)
 		(stroke
@@
 	(wire
 		(pts
-			(xy 69.85 190.5) (xy 73.66 190.5)
+			(xy 67.31 190.5) (xy 73.66 190.5)
 		)
 		(stroke
@@
 		)
 	)
-	(label "S2"
-		(at 44.45 190.5 0)
+	(label "S2_MP"
+		(at 41.91 190.5 0)
 		(fields_autoplaced yes)
 		(effects
@@
 		)
 	)
-	(label "S1"
-		(at 69.85 187.96 0)
+	(label "S1_RF"
+		(at 67.31 187.96 0)
 		(fields_autoplaced yes)
 		(effects
@@
 		)
 	)
-	(label "S1"
-		(at 44.45 187.96 0)
+	(label "S1_MP"
+		(at 41.91 187.96 0)
 		(fields_autoplaced yes)
 		(effects
@@
 		)
 	)
-	(label "S2"
-		(at 69.85 190.5 0)
-		(fields_autoplaced yes)
-		(effects
+	(label "S2_RF"
+		(at 67.31 190.5 0)
+		(fields_autoplaced yes)
+		(effects

Commit message: fixed ribbon connectors and S1 & S2
Connections:
- net S1_MP: now also U1.10 (PA0)
- net S1_RF: now also U1.27 (PB14)
- net S2_MP: now also U1.11 (PA1)
- net S2_RF: now also U1.28 (PB15)
- no-connect marks 24 -> 20
Changed lines of the file:
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@@
 	)
 	(no_connect
-		(at 86.36 127)
-	)
-	(no_connect
 		(at 364.49 125.73)
 	)
@@
 	)
 	(no_connect
-		(at 119.38 93.98)
-	)
-	(no_connect
 		(at 206.502 70.612)
 	)
@@
 	)
 	(no_connect
-		(at 119.38 91.44)
-	)
-	(no_connect
 		(at 86.36 86.36)
 	)
@@
 		(at 223.266 229.87)
 	)
-	(no_connect
-		(at 86.36 129.54)
-	)
 	(wire
 		(pts
@@
 	(wire
 		(pts
+			(xy 78.74 127) (xy 86.36 127)
+		)
+		(stroke
+			(width 0)
+			(type default)
+		)
+	)
+	(wire
+		(pts
 			(xy 72.39 200.66) (xy 73.66 200.66)
 		)
@@
 	(wire
 		(pts
+			(xy 78.74 129.54) (xy 86.36 129.54)
+		)
+		(stroke
+			(width 0)
+			(type default)
+		)
+	)
+	(wire
+		(pts
 			(xy 204.978 33.274) (xy 204.978 35.814)
 		)
@@
 	(wire
 		(pts
+			(xy 119.38 93.98) (xy 127 93.98)
+		)
+		(stroke
+			(width 0)
+			(type default)
+		)
+	)
+	(wire
+		(pts
 			(xy 119.38 104.14) (xy 124.968 104.14)
 		)
@@
 	(wire
 		(pts
+			(xy 119.38 91.44) (xy 127 91.44)
+		)
+		(stroke
+			(width 0)
+			(type default)
+		)
+	)
+	(wire
+		(pts
 			(xy 205.74 62.992) (xy 206.502 62.992)
 		)
@@
 		)
 	)
+	(label "S1_MP"
+		(at 127 91.44 180)
+		(fields_autoplaced yes)
+		(effects
+			(font
+				(size 1.27 1.27)
+			)
+			(justify right bottom)
+		)
+	)
 	(label "TX_GPS"
 		(at 320.04 130.81 0)
@@
 		)
 	)
+	(label "S2_MP"
+		(at 127 93.98 180)
+		(fields_autoplaced yes)
+		(effects
+			(font
+				(size 1.27 1.27)
+			)
+			(justify right bottom)
+		)
+	)
 	(label "TX_GPS"
 		(at 128.27 99.06 180)
@@
 		)
 	)
+	(label "S1_RF"
+		(at 78.74 127 0)
+		(fields_autoplaced yes)
+		(effects
+			(font
+				(size 1.27 1.27)
+			)
+			(justify left bottom)
+		)
+	)
 	(label "S2_RF"
 		(at 67.31 190.5 0)
@@
 		)
 	)
+	(label "S2_RF"
+		(at 78.74 129.54 0)
+		(fields_autoplaced yes)
+		(effects
+			(font
+				(size 1.27 1.27)
+			)
+			(justify left bottom)
+		)
+	)

Commit message: added most part numbers
Parts:
- J1: LCSC Part (none) -> C3025061
- J3, J6: LCSC Part (none) -> C505273
- R12, R13: LCSC Part C25906 -> C119339
- U3: LCSC Part (none) -> C83291
Changed lines of the file:
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@@
 			)
 		)
+		(property "LCSC Part" "C505273"
+			(at 53.34 190.5 0)
+			(effects
+				(font
+					(size 1.27 1.27)
+				)
+				(hide yes)
+			)
+		)
 		(pin "4"
 		)
@@
 			)
 		)
-		(property "LCSC Part" "C25906"
+		(property "LCSC Part" "C119339"
 			(at 73.66 114.3 0)
 			(effects
@@
 			)
 		)
+		(property "LCSC Part" "C3025061"
+			(at 252.73 113.03 0)
+			(effects
+				(font
+					(size 1.27 1.27)
+				)
+				(hide yes)
+			)
+		)
 		(pin "1"
 		)
@@
 			)
 		)
+		(property "LCSC Part" "C505273"
+			(at 78.74 190.5 0)
+			(effects
+				(font
+					(size 1.27 1.27)
+				)
+				(hide yes)
+			)
+		)
 		(pin "4"
 		)
@@
 			)
 		)
-		(property "LCSC Part" "C25906"
+		(property "LCSC Part" "C119339"
 			(at 73.66 111.76 0)
 			(effects
@@
 				(hide yes)
 			)
+		)
+		(property "LCSC Part" "C83291"
+			(at 334.01 60.96 0)
+			(effects
+				(font
+					(size 1.27 1.27)
+				)
+				(hide yes)
+			)

Commit message: added tentative external i2c connectors
Parts:
- added J7, J8: Conn_01x04_Pin, Connector_JST:JST_SH_BM04B-SRSS-TB_1x04-1MP_P1.00mm_Vertical, symbol Connector:Conn_01x04_Pin
Connections:
- net +3.3V: now also J7.1 (Pin_1), J8.1 (Pin_1)
- net GND: now also J7.4 (Pin_4), J8.4 (Pin_4)
- net SCL: now also J7.3 (Pin_3), J8.3 (Pin_3)
- net SDA: now also J7.2 (Pin_2), J8.2 (Pin_2)
Other:
- note added: "Ext. I2C"
- moved on the sheet: J1, J4, J5

Commit message: fixed motor conn. i2c and external i2c conn.s, changed PNs, added models
new PN for Y2, added 3D models for BMP, Antenna, and ext. i2c connectors.
Parts:
- added R15, R16: 4.7k, Resistor_SMD:R_0402_1005Metric, symbol Device:R
- Y2: value 32.768Mhz -> 32.768kHz; LCSC Part C907540 -> C32346
Connections:
- net +3.3V: now also R15.2, R16.2; no longer J3.5 (Pin_5), J3.6 (Pin_6), U1.21 (PB10), U1.39 (PB3)
- new net MOTOR_SCL: J3.6 (Pin_6), R16.1, U1.21 (PB10)
- new net MOTOR_SDA: J3.5 (Pin_5), R15.1, U1.39 (PB3)
Other:
- moved on the sheet: R12, R13
Changed lines of the file:
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@@
 	)
 	(junction
-		(at 67.31 113.03)
+		(at 63.5 113.03)
 		(diameter 0)
 		(color 0 0 0 0)
@@
 	(wire
 		(pts
-			(xy 41.91 129.54) (xy 54.61 129.54)
+			(xy 41.91 129.54) (xy 43.18 129.54)
 		)
 		(stroke
@@
 	(wire
 		(pts
-			(xy 77.47 114.3) (xy 86.36 114.3)
+			(xy 73.66 114.3) (xy 86.36 114.3)
 		)
 		(stroke
@@
 	(wire
 		(pts
-			(xy 67.31 114.3) (xy 69.85 114.3)
+			(xy 63.5 114.3) (xy 66.04 114.3)
 		)
 		(stroke
@@
 	(wire
 		(pts
-			(xy 54.61 125.73) (xy 41.91 125.73)
+			(xy 62.23 125.73) (xy 50.8 125.73)
 		)
 		(stroke
@@
 	(wire
 		(pts
+			(xy 50.8 129.54) (xy 62.23 129.54)
+		)
+		(stroke
+			(width 0)
+			(type default)
+		)
+	)
+	(wire
+		(pts
 			(xy 311.15 100.33) (xy 311.15 101.6)
 		)
@@
 	(wire
 		(pts
-			(xy 67.31 111.76) (xy 67.31 113.03)
+			(xy 63.5 111.76) (xy 63.5 113.03)
 		)
 		(stroke
@@
 	(wire
 		(pts
-			(xy 77.47 111.76) (xy 86.36 111.76)
+			(xy 73.66 111.76) (xy 86.36 111.76)
 		)
 		(stroke
@@
 	(wire
 		(pts
-			(xy 67.31 113.03) (xy 67.31 114.3)
+			(xy 63.5 113.03) (xy 63.5 114.3)
 		)
 		(stroke
@@
 	(wire
 		(pts
-			(xy 67.31 111.76) (xy 69.85 111.76)
+			(xy 63.5 111.76) (xy 66.04 111.76)
 		)
 		(stroke
@@
 	(wire
 		(pts
+			(xy 43.18 125.73) (xy 41.91 125.73)
+		)
+		(stroke
+			(width 0)
+			(type default)
+		)
+	)
+	(wire
+		(pts
 			(xy 64.77 102.87) (xy 64.77 105.41)
 		)
@@
 	(wire
 		(pts
-			(xy 67.31 113.03) (xy 64.77 113.03)
+			(xy 63.5 113.03) (xy 60.96 113.03)
 		)
 		(stroke
@@
 	)
 	(label "MOTOR_SDA"
-		(at 54.61 125.73 180)
+		(at 62.23 125.73 180)
 		(fields_autoplaced yes)
 		(effects
@@
 	)
 	(label "MOTOR_SCL"
-		(at 54.61 129.54 180)
+		(at 62.23 129.54 180)
 		(fields_autoplaced yes)
 		(effects
@@
 	)
 	(symbol
+		(lib_id "Device:R")
+		(at 46.99 125.73 270)
+		(unit 1)
+		(exclude_from_sim no)
+		(in_bom yes)
+		(on_board yes)
+		(dnp no)
+		(property "Reference" "R15"
+			(at 46.99 123.698 90)
+			(effects
+				(font
+					(size 1.27 1.27)
+				)
+			)
+		)
+		(property "Value" "4.7k"
+			(at 46.99 125.73 90)
+			(effects
+				(font
+					(size 1.27 1.27)
+				)
+			)
+		)
+		(property "Footprint" "Resistor_SMD:R_0402_1005Metric"
+			(at 46.99 123.952 90)
+			(effects
+				(font
+					(size 1.27 1.27)
+				)
+				(hide yes)
+			)
+		)
+		(property "Datasheet" "~"
+			(at 46.99 125.73 0)
+			(effects
+				(font
+					(size 1.27 1.27)
+				)
+				(hide yes)
+			)
+		)
+		(property "Description" ""
+			(at 46.99 125.73 0)
+			(effects
+				(font
+					(size 1.27 1.27)
+				)
+				(hide yes)
+			)
+		)
+		(property "LCSC Part" "C119339"
+			(at 46.99 125.73 0)
+			(effects
+				(font
+					(size 1.27 1.27)
+				)
+				(hide yes)
+			)
+		)
+		(pin "1"
+		)
+		(pin "2"
+		)
+		(instances
+			(project "ARES_FC"
+				(path "/449acbee-2eeb-4316-a8e9-c26dd430524e"
+					(reference "R15")
+					(unit 1)
+				)
+			)
+		)
+	)
+	(symbol
 		(lib_id "power:GND")
 		(at 140.208 48.514 0)
@@
 	(symbol
 		(lib_id "Device:R")
-		(at 73.66 114.3 270)
+		(at 69.85 114.3 270)
 		(unit 1)
 		(exclude_from_sim no)
@@
 		(dnp no)
 		(property "Reference" "R13"
-			(at 73.66 116.586 90)
+			(at 69.85 116.586 90)
 			(effects
 				(font
@@
 		)
 		(property "Value" "4.7k"
-			(at 73.66 114.3 90)
+			(at 69.85 114.3 90)
 			(effects
 				(font
@@
 		)
 		(property "Footprint" "Resistor_SMD:R_0402_1005Metric"
-			(at 73.66 112.522 90)
+			(at 69.85 112.522 90)
 			(effects
 				(font
@@
 		)
 		(property "Datasheet" "~"
-			(at 73.66 114.3 0)
+			(at 69.85 114.3 0)
 			(effects
 				(font
@@
 		)
 		(property "Description" ""
-			(at 73.66 114.3 0)
+			(at 69.85 114.3 0)
 			(effects
 				(font
@@
 		)
 		(property "LCSC Part" "C119339"
-			(at 73.66 114.3 0)
+			(at 69.85 114.3 0)
 			(effects
 				(font
@@
 		(lib_name "+3.3V_1")
 		(lib_id "power:+3.3V")
-		(at 64.77 113.03 90)
+		(at 60.96 113.03 90)
 		(unit 1)
 		(exclude_from_sim no)
@@
 		(fields_autoplaced yes)
 		(property "Reference" "#PWR023"
-			(at 68.58 113.03 0)
+			(at 64.77 113.03 0)
 			(effects
 				(font
@@
 		)
 		(property "Value" "+3.3V"
-			(at 60.96 113.0299 90)
+			(at 57.15 113.0299 90)
 			(effects
 				(font
@@
 		)
 		(property "Footprint" ""
-			(at 64.77 113.03 0)
+			(at 60.96 113.03 0)
 			(effects
 				(font
@@
 		)
 		(property "Datasheet" ""
-			(at 64.77 113.03 0)
+			(at 60.96 113.03 0)
 			(effects
 				(font
@@
 		)
 		(property "Description" "Power symbol creates a global label with name \"+3.3V\""
-			(at 64.77 113.03 0)
+			(at 60.96 113.03 0)
 			(effects
 				(font
@@
 			)
 		)
-		(property "Value" "32.768Mhz"
+		(property "Value" "32.768kHz"
 			(at 349.7834 199.3142 90)
 			(effects
@@
 			)
 		)
-		(property "LCSC Part" "C907540"
+		(property "LCSC Part" " C32346"
 			(at 346.456 197.612 0)
 			(effects
@@
 	(symbol
 		(lib_id "Device:R")
+		(at 46.99 129.54 270)
+		(unit 1)
+		(exclude_from_sim no)
+		(in_bom yes)
+		(on_board yes)
+		(dnp no)
+		(property "Reference" "R16"
+			(at 46.99 131.826 90)
+			(effects
+				(font
+					(size 1.27 1.27)
+				)
+			)
+		)
+		(property "Value" "4.7k"
+			(at 46.99 129.54 90)
+			(effects
+				(font
+					(size 1.27 1.27)
+				)
+			)
+		)
+		(property "Footprint" "Resistor_SMD:R_0402_1005Metric"
+			(at 46.99 127.762 90)
+			(effects
+				(font
+					(size 1.27 1.27)
+				)
+				(hide yes)
+			)
+		)
+		(property "Datasheet" "~"
+			(at 46.99 129.54 0)
+			(effects
+				(font
+					(size 1.27 1.27)
+				)
+				(hide yes)
+			)
+		)
+		(property "Description" ""
+			(at 46.99 129.54 0)
+			(effects
+				(font
+					(size 1.27 1.27)
+				)
+				(hide yes)
+			)
+		)
+		(property "LCSC Part" "C119339"
+			(at 46.99 129.54 0)
+			(effects
+				(font
+					(size 1.27 1.27)
+				)
+				(hide yes)
+			)
+		)
+		(pin "1"
+		)
+		(pin "2"
+		)
+		(instances
+			(project "ARES_FC"
+				(path "/449acbee-2eeb-4316-a8e9-c26dd430524e"
+					(reference "R16")
+					(unit 1)
+				)
+			)
+		)
+	)
+	(symbol
+		(lib_id "Device:R")
 		(at 137.668 193.04 0)
 		(unit 1)
@@
 	(symbol
 		(lib_id "Device:R")
-		(at 73.66 111.76 270)
+		(at 69.85 111.76 270)
 		(mirror x)
 		(unit 1)
@@
 		(dnp no)
 		(property "Reference" "R12"
-			(at 73.66 109.474 90)
+			(at 69.85 109.474 90)
 			(effects
 				(font
@@
 		)
 		(property "Value" "4.7k"
-			(at 73.66 111.76 90)
+			(at 69.85 111.76 90)
 			(effects
 				(font
@@
 		)
 		(property "Footprint" "Resistor_SMD:R_0402_1005Metric"
-			(at 73.66 113.538 90)
+			(at 69.85 113.538 90)
 			(effects
 				(font
@@
 		)
 		(property "Datasheet" "~"
-			(at 73.66 111.76 0)
+			(at 69.85 111.76 0)
 			(effects
 				(font
@@
 		)
 		(property "Description" ""
-			(at 73.66 111.76 0)
+			(at 69.85 111.76 0)
 			(effects
 				(font
@@
 		)
 		(property "LCSC Part" "C119339"
-			(at 73.66 111.76 0)
+			(at 69.85 111.76 0)
 			(effects
 				(font
