File: Hardware/PullTab/pulltab.kicad_sch (KiCad schematic)
At the start: 9 parts, among them J1 Switch_Junction, J2 GND_IN, J4 VBAT_IN, J5 Switch_NC, J6 VBAT_OUT, J7 GND_OUT, Q1 NMOS

Commit message: fixed pulltab mosfet pin orientation added cad
Connections:
- net at J7.1 (Pin_1): now also Q1.2 (D); no longer Q1.1 (D)
- net at J1.1 (Pin_1), R1.1: now also Q1.1 (G); no longer Q1.2 (G)
